Commit message: draft submission for SnC as custom ros package

File: Sensors_n_Control_Only/tm5_custom/description/urdf/tm.gazebo.xacro (robot description, xacro)
@@ -39,7 +39,7 @@
             <pose> 0 0 0 0 ${pi/2} ${pi/2} </pose>
             <visualize>true</visualize>
-            <update_rate>10</update_rate>
+            <update_rate>30</update_rate>
             <camera>
-                <horizontal_fov>1.089</horizontal_fov>
+                <horizontal_fov>0.988987</horizontal_fov>
                 <image>
                     <format>R8G8B8</format>
@@ -51,4 +51,13 @@
                     <far>4.0</far>
                 </clip>
+                <!--
+                <distortion>
+                  <k1>-0.23880386371963863</k1>
+                  <k2>-0.7214320219570768</k2>
+                  <k3>1.941908386385502 </k3>
+                  <p1>-0.00037858100167365054</p1>
+                  <p2>0.0025032179171072936</p2>
+                  <center>0.27903 0.197760</center>
+                </distortion>-->
             </camera>
             <plugin name="camera_controller" filename="libgazebo_ros_camera.so">

File: Sensors_n_Control_Only/tm5_custom/description/urdf/user_defined_tm5-700.urdf.xacro (robot description, xacro)
@@ -68,11 +68,11 @@
     <visual>
       <geometry>
-        <mesh filename="$(find tm5_custom)/description/meshes/visual/tm5-base.${format}" />
-      </geometry>
-      <material name="${color}" />
-    </visual>
-    <collision>
-      <geometry>
-        <mesh filename="$(find tm5_custom)/description/meshes/collision/tm5-base_c.stl" />
+        <mesh filename="package://tm5_custom/description/meshes/visual/tm5-base.${format}" />
+      </geometry>
+      <material name="${color}" />
+    </visual>
+    <collision>
+      <geometry>
+        <mesh filename="package://tm5_custom/description/meshes/collision/tm5-base_c.stl" />
       </geometry>
     </collision>
@@ -97,11 +97,11 @@
     <visual>
       <geometry>
-        <mesh filename="$(find tm5_custom)/description/meshes/visual/tmr_400w_01.${format}" />
-      </geometry>
-      <material name="${color}" />
-    </visual>
-    <collision>
-      <geometry>
-        <mesh filename="$(find tm5_custom)/description/meshes/collision/tmr_400w_01_c.stl" />
+        <mesh filename="package://tm5_custom/description/meshes/visual/tmr_400w_01.${format}" />
+      </geometry>
+      <material name="${color}" />
+    </visual>
+    <collision>
+      <geometry>
+        <mesh filename="package://tm5_custom/description/meshes/collision/tmr_400w_01_c.stl" />
       </geometry>
     </collision>
@@ -127,11 +127,11 @@
     <visual>
       <geometry>
-        <mesh filename="$(find tm5_custom)/description/meshes/visual/tm5-700_arm1.${format}" />
-      </geometry>
-      <material name="${color}" />
-    </visual>
-    <collision>
-      <geometry>
-        <mesh filename="$(find tm5_custom)/description/meshes/collision/tm5-700_arm1_c.stl" />
+        <mesh filename="package://tm5_custom/description/meshes/visual/tm5-700_arm1.${format}" />
+      </geometry>
+      <material name="${color}" />
+    </visual>
+    <collision>
+      <geometry>
+        <mesh filename="package://tm5_custom/description/meshes/collision/tm5-700_arm1_c.stl" />
       </geometry>
     </collision>
@@ -157,11 +157,11 @@
     <visual>
       <geometry>
-        <mesh filename="$(find tm5_custom)/description/meshes/visual/tm5-700_arm2.${format}" />
-      </geometry>
-      <material name="${color}" />
-    </visual>
-    <collision>
-      <geometry>
-        <mesh filename="$(find tm5_custom)/description/meshes/collision/tm5-700_arm2_c.stl" />
+        <mesh filename="package://tm5_custom/description/meshes/visual/tm5-700_arm2.${format}" />
+      </geometry>
+      <material name="${color}" />
+    </visual>
+    <collision>
+      <geometry>
+        <mesh filename="package://tm5_custom/description/meshes/collision/tm5-700_arm2_c.stl" />
       </geometry>
     </collision>
@@ -187,11 +187,11 @@
     <visual>
       <geometry>
-        <mesh filename="$(find tm5_custom)/description/meshes/visual/tmr_100w_01.${format}" />
-      </geometry>
-      <material name="${color}" />
-    </visual>
-    <collision>
-      <geometry>
-        <mesh filename="$(find tm5_custom)/description/meshes/collision/tmr_100w_01_c.stl" />
+        <mesh filename="package://tm5_custom/description/meshes/visual/tmr_100w_01.${format}" />
+      </geometry>
+      <material name="${color}" />
+    </visual>
+    <collision>
+      <geometry>
+        <mesh filename="package://tm5_custom/description/meshes/collision/tmr_100w_01_c.stl" />
       </geometry>
     </collision>
@@ -217,11 +217,11 @@
     <visual>
       <geometry>
-        <mesh filename="$(find tm5_custom)/description/meshes/visual/tmr_100w_02.${format}" />
-      </geometry>
-      <material name="${color}" />
-    </visual>
-    <collision>
-      <geometry>
-        <mesh filename="$(find tm5_custom)/description/meshes/collision/tmr_100w_02_c.stl" />
+        <mesh filename="package://tm5_custom/description/meshes/visual/tmr_100w_02.${format}" />
+      </geometry>
+      <material name="${color}" />
+    </visual>
+    <collision>
+      <geometry>
+        <mesh filename="package://tm5_custom/description/meshes/collision/tmr_100w_02_c.stl" />
       </geometry>
     </collision>
@@ -247,5 +247,5 @@
     <visual>
       <geometry>
-        <mesh filename="$(find tm5_custom)/description/meshes/visual/tmr_ee.${format}" />
+        <mesh filename="package://tm5_custom/description/meshes/visual/tmr_ee.${format}" />
       </geometry>
       <material name="${color}" />
@@ -254,5 +254,5 @@
     <collision>
       <geometry>
-        <mesh filename="$(find tm5_custom)/description/meshes/collision/tmr_ee_c.stl" />
+        <mesh filename="package://tm5_custom/description/meshes/collision/tmr_ee_c.stl" />
       </geometry>
     </collision>
@@ -279,5 +279,5 @@
   <visual>
         <geometry>
-            <mesh filename="$(find tm5_custom)/description/meshes/visual/endEffectorFixed.stl" />
+            <mesh filename="package://tm5_custom/description/meshes/visual/endEffectorFixed.stl" />
         </geometry>
         <!-- Optional: Add material for the visual representation of your tool -->
@@ -286,5 +286,5 @@
     <collision>
         <geometry>
-            <mesh filename="$(find tm5_custom)/description/meshes/collision/endEffectorFixed.stl" />
+            <mesh filename="package://tm5_custom/description/meshes/collision/endEffectorFixed.stl" />
         </geometry>
     </collision>
